Commit message: xarco include and gazebo launch

File: src/m2wr_description/urdf/m2wr.xacro (robot description, xacro)
@@ -1,37 +1,6 @@
 <?xml version="1.0" ?>
 <robot name="m2wr" xmlns:xacro="https://www.ros.org/wiki/xacro" >
-  <material name="black">
-    <color rgba="0.0 0.0 0.0 1.0"/>
-  </material>
-  <material name="blue">
-    <color rgba="0.203125 0.23828125 0.28515625 1.0"/>
-  </material>
-  <material name="green">
-    <color rgba="0.0 0.8 0.0 1.0"/>
-  </material>
-  <material name="grey">
-    <color rgba="0.2 0.2 0.2 1.0"/>
-  </material>
-  <material name="orange">
-    <color rgba="1.0 0.423529411765 0.0392156862745 1.0"/>
-  </material>
-  <material name="brown">
-    <color rgba="0.870588235294 0.811764705882 0.764705882353 1.0"/>
-  </material>
-  <material name="red">
-    <color rgba="0.80078125 0.12890625 0.1328125 1.0"/>
-  </material>
-  <material name="white">
-    <color rgba="1.0 1.0 1.0 1.0"/>
-  </material>
-  <gazebo reference="link_chassis">
-    <material>Gazebo/Orange</material>
-  </gazebo>
-  <gazebo reference="link_left_wheel">
-    <material>Gazebo/Blue</material>
-  </gazebo>
-  <gazebo reference="link_right_wheel">
-    <material>Gazebo/Blue</material>
-  </gazebo>
+    <xacro:include filename="$(find m2wr_description)/urdf/gazebo.xacro"/>
+    <xacro:include filename="$(find m2wr_description)/urdf/materials.xacro"/>
   <link name="link_chassis">
     <!-- pose and inertial -->

Commit message: fix: add xacro ns to macro tag

File: src/m2wr_description/urdf/m2wr.xacro (robot description, xacro)
@@ -1,3 +1,2 @@
-<!-- https://bitbucket.org/theconstructcore/box_car/src/foxy/box_car_description/robot/ -->
 <?xml version="1.0" ?>
 <robot name="m2wr"

File: src/m2wr_description/urdf/macros.xacro (robot description, xacro)
@@ -1,5 +1,5 @@
 <?xml version="1.0"?>
-<robot>
-    <macro name="link_wheel" params="name">
+<robot xmlns:xacro="https://www.ros.org/wiki/xacro">
+    <xacro:macro name="link_wheel" params="name">
         <link name="${name}">
             <inertial>
@@ -21,6 +21,6 @@
             </visual>
         </link>
-    </macro>
-    <macro name="joint_wheel" params="name child origin_xyz">
+    </xacro:macro>
+    <xacro:macro name="joint_wheel" params="name child origin_xyz">
       <joint name="${name}" type="continuous">
         <origin rpy="0 0 0" xyz="${origin_xyz}"/>
@@ -31,4 +31,4 @@
         <joint_properties damping="1.0" friction="1.0"/>
       </joint>
-    </macro>
+    </xacro:macro>
 </robot>
