Commit message: fix: gazebo diff plugin

File: src/m2wr_description/urdf/gazebo.xacro (robot description, xacro)
@@ -13,16 +13,20 @@
     <gazebo>
         <plugin filename="libgazebo_ros_diff_drive.so" name="differential_drive_controller">
+            <ros>
+                <namespace>/m2wr</namespace>
+            </ros>
             <legacyMode>false</legacyMode>
             <alwaysOn>true</alwaysOn>
             <updateRate>20</updateRate>
-            <leftJoint>joint_left_wheel</leftJoint>
-            <rightJoint>joint_right_wheel</rightJoint>
-            <wheelSeparation>0.2</wheelSeparation>
-            <wheelDiameter>0.2</wheelDiameter>
+            <left_joint>joint_left_wheel</left_joint>
+            <right_joint>joint_right_wheel</right_joint>
+            <wheel_separation>0.2</wheel_separation>
+            <wheel_diameter>0.2</wheel_diameter>
             <torque>0.1</torque>
             <commandTopic>cmd_vel</commandTopic>
-            <odometryTopic>odom</odometryTopic>
-            <odometryFrame>odom</odometryFrame>
-            <robotBaseFrame>link_chassis</robotBaseFrame>
+            <publish_odom>true</publish_odom>
+            <publish_odom_tf>true</publish_odom_tf>
+            <odometry_frame>odom</odometry_frame>
+            <robot_base_frame>link_chassis</robot_base_frame>
         </plugin>
     </gazebo>

File: src/m2wr_description/urdf/m2wr.xacro (robot description, xacro)
@@ -1,6 +1,9 @@
+<!-- https://bitbucket.org/theconstructcore/box_car/src/foxy/box_car_description/robot/ -->
 <?xml version="1.0" ?>
-<robot name="m2wr" xmlns:xacro="https://www.ros.org/wiki/xacro" >
-    <xacro:include filename="$(find m2wr_description)/urdf/gazebo.xacro"/>
-    <xacro:include filename="$(find m2wr_description)/urdf/materials.xacro"/>
+<robot name="m2wr"
+  xmlns:xacro="https://www.ros.org/wiki/xacro">
+  <xacro:include filename="$(find m2wr_description)/urdf/gazebo.xacro"/>
+  <xacro:include filename="$(find m2wr_description)/urdf/materials.xacro"/>
+  <xacro:include filename="$(find m2wr_description)/urdf/macros.xacro" />
   <link name="link_chassis">
     <!-- pose and inertial -->
@@ -11,4 +14,5 @@
       <inertia ixx="0.0395416666667" ixy="0" ixz="0" iyy="0.106208333333" iyz="0" izz="0.106208333333"/>
     </inertial>
+    <!-- body -->
     <collision name="collision_chassis">
       <geometry>
@@ -46,62 +50,8 @@
       </geometry>
     </visual>
-    </link>
-  <!-- Create wheel right -->
-  <link name="link_right_wheel">
-    <inertial>
-      <mass value="0.2"/>
-      <origin rpy="0 1.5707 1.5707" xyz="0 0 0"/>
-      <inertia ixx="0.00052666666" ixy="0" ixz="0" iyy="0.00052666666" iyz="0" izz="0.001"/>
-    </inertial>
-    <collision name="link_right_wheel_collision">
-      <origin rpy="0 1.5707 1.5707" xyz="0 0 0" />
-      <geometry>
-        <cylinder length="0.04" radius="0.1"/>
-      </geometry>
-    </collision>
-    <visual name="link_right_wheel_visual">
-      <origin rpy="0 1.5707 1.5707" xyz="0 0 0"/>
-      <geometry>
-        <cylinder length="0.04" radius="0.1"/>
-      </geometry>
-    </visual>
   </link>
-  <!--   Joint for right wheel  -->
-  <joint name="joint_right_wheel" type="continuous">
-    <origin rpy="0 0 0" xyz="-0.05 0.15 0"/>
-    <child link="link_right_wheel" />
-    <parent link="link_chassis"/>
-    <axis rpy="0 0 0" xyz="0 1 0"/>
-    <limit effort="10000" velocity="1000"/>
-    <joint_properties damping="1.0" friction="1.0" />
-  </joint>
-  <!-- Left Wheel link -->
-  <link name="link_left_wheel">
-    <inertial>
-      <mass value="0.2"/>
-      <origin rpy="0 1.5707 1.5707" xyz="0 0 0"/>
-      <inertia ixx="0.00052666666" ixy="0" ixz="0" iyy="0.00052666666" iyz="0" izz="0.001"/>
-    </inertial>
-    <collision name="link_left_wheel_collision">
-      <origin rpy="0 1.5707 1.5707" xyz="0 0 0" />
-      <geometry>
-        <cylinder length="0.04" radius="0.1"/>
-      </geometry>
-    </collision>
-    <visual name="link_left_wheel_visual">
-      <origin rpy="0 1.5707 1.5707" xyz="0 0 0"/>
-      <geometry>
-        <cylinder length="0.04" radius="0.1"/>
-      </geometry>
-    </visual>
-  </link>
-  <!--   Joint for right wheel  -->
-  <joint name="joint_left_wheel" type="continuous">
-    <origin rpy="0 0 0" xyz="-0.05 -0.15 0"/>
-    <child link="link_left_wheel" />
-    <parent link="link_chassis"/>
-    <axis rpy="0 0 0" xyz="0 1 0"/>
-    <limit effort="10000" velocity="1000"/>
-    <joint_properties damping="1.0" friction="1.0" />
-  </joint>
+  <xacro:link_wheel name="link_right_wheel" />
+  <xacro:joint_wheel name="joint_right_wheel" child="link_right_wheel" origin_xyz="-0.05 0.15 0" />
+  <xacro:link_wheel name="link_left_wheel" />
+  <xacro:joint_wheel name="joint_left_wheel" child="link_left_wheel" origin_xyz="-0.05 -0.15 0" />
 </robot>

Commit message: feat: add gz world and add ray sensor

File: src/m2wr_description/urdf/gazebo.xacro (robot description, xacro)
@@ -34,3 +34,37 @@
         </plugin>
     </gazebo>
+    <gazebo reference="sensor_laser">
+        <sensor type="ray" name="head_hokuyo_sensor">
+            <pose>0 0 0 0 0 0</pose>
+            <visualize>false</visualize>
+            <update_rate>20</update_rate>
+            <ray>
+                <scan>
+                    <horizontal>
+                        <samples>720</samples>
+                        <resolution>1</resolution>
+                        <min_angle>-1.570796</min_angle>
+                        <max_angle>1.570796</max_angle>
+                    </horizontal>
+                </scan>
+                <range>
+                    <min>0.10</min>
+                    <max>10.0</max>
+                    <resolution>0.01</resolution>
+                </range>
+                <noise>
+                    <type>gaussian</type>
+                    <mean>0.0</mean>
+                    <stddev>0.01</stddev>
+                </noise>
+            </ray>
+            <plugin name="gazebo_ros_head_hokuyo_controller" filename="libgazebo_ros_ray_sensor.so">
+                <ros>
+                    <namespace>/m2wr</namespace>
+                    <argument>~/out:=scan</argument>
+                </ros>
+                <output_type>sensor_msgs/LaserScan</output_type>
+            </plugin>
+        </sensor>
+    </gazebo>
 </robot>

File: src/m2wr_description/urdf/m2wr.xacro (robot description, xacro)
@@ -50,4 +50,30 @@
     </visual>
   </link>
+  <!-- laser -->
+  <link name="sensor_laser">
+    <inertial>
+      <origin xyz="0 0 0" rpy="0 0 0" />
+      <mass value="1" />
+      <xacro:cylinder_inertia mass="1" r="0.05" l="0.1" />
+    </inertial>
+    <visual>
+      <origin xyz="0 0 0" rpy="0 0 0" />
+      <geometry>
+        <cylinder radius="0.05" length="0.1"/>
+      </geometry>
+      <material name="white" />
+    </visual>
+    <collision>
+      <origin xyz="0 0 0" rpy="0 0 0"/>
+      <geometry>
+        <cylinder radius="0.05" length="0.1"/>
+      </geometry>
+    </collision>
+  </link>
+  <joint name="joint_sensor_laser" type="fixed">
+    <origin xyz="0.15 0 0.05" rpy="0 0 0"/>
+    <parent link="link_chassis"/>
+    <child link="sensor_laser"/>
+  </joint>
   <xacro:link_wheel name="link_right_wheel" />
   <xacro:joint_wheel name="joint_right_wheel" child="link_right_wheel" origin_xyz="-0.05 0.15 0" />

File: src/m2wr_description/urdf/macros.xacro (robot description, xacro)
@@ -1,34 +1,37 @@
 <?xml version="1.0"?>
 <robot xmlns:xacro="https://www.ros.org/wiki/xacro">
-    <xacro:macro name="link_wheel" params="name">
-        <link name="${name}">
-            <inertial>
-              <mass value="0.2"/>
-              <origin rpy="0 1.5707 1.5707" xyz="0 0 0"/>
-              <inertia ixx="0.000526666666667" ixy="0" ixz="0" iyy="0.000526666666667" iyz="0" izz="0.001"/>
-            </inertial>
-            <collision name="link_right_wheel_collision">
-              <origin rpy="0 1.5707 1.5707" xyz="0 0 0"/>
-              <geometry>
-                <cylinder length="0.04" radius="0.1"/>
-              </geometry>
-            </collision>
-            <visual name="${name}_visual">
-              <origin rpy="0 1.5707 1.5707" xyz="0 0 0"/>
-              <geometry>
-                <cylinder length="0.04" radius="0.1"/>
-              </geometry>
-            </visual>
-        </link>
-    </xacro:macro>
-    <xacro:macro name="joint_wheel" params="name child origin_xyz">
-      <joint name="${name}" type="continuous">
-        <origin rpy="0 0 0" xyz="${origin_xyz}"/>
-        <child link="${child}"/>
-        <parent link="link_chassis"/>
-        <axis rpy="0 0 0" xyz="0 1 0"/>
-        <limit effort="10000" velocity="1000"/>
-        <joint_properties damping="1.0" friction="1.0"/>
-      </joint>
-    </xacro:macro>
+  <xacro:macro name="link_wheel" params="name">
+    <link name="${name}">
+      <inertial>
+        <mass value="0.2"/>
+        <origin rpy="0 1.5707 1.5707" xyz="0 0 0"/>
+        <inertia ixx="0.000526666666667" ixy="0" ixz="0" iyy="0.000526666666667" iyz="0" izz="0.001"/>
+      </inertial>
+      <collision name="link_right_wheel_collision">
+        <origin rpy="0 1.5707 1.5707" xyz="0 0 0"/>
+        <geometry>
+          <cylinder length="0.04" radius="0.1"/>
+        </geometry>
+      </collision>
+      <visual name="${name}_visual">
+        <origin rpy="0 1.5707 1.5707" xyz="0 0 0"/>
+        <geometry>
+          <cylinder length="0.04" radius="0.1"/>
+        </geometry>
+      </visual>
+    </link>
+  </xacro:macro>
+  <xacro:macro name="cylinder_inertia" params="mass r l">
+    <inertia ixx="${mass*(3*r*r+l*l)/12}" ixy = "0" ixz = "0" iyy="${mass*(3*r*r+l*l)/12}" iyz = "0" izz="${mass*(r*r)/2}" />
+  </xacro:macro>
+  <xacro:macro name="joint_wheel" params="name child origin_xyz">
+    <joint name="${name}" type="continuous">
+      <origin rpy="0 0 0" xyz="${origin_xyz}"/>
+      <child link="${child}"/>
+      <parent link="link_chassis"/>
+      <axis rpy="0 0 0" xyz="0 1 0"/>
+      <limit effort="10000" velocity="1000"/>
+      <joint_properties damping="1.0" friction="1.0"/>
+    </joint>
+  </xacro:macro>
 </robot>
